File: SSI Balloon Summer PCB/GPS.kicad_sch (KiCad schematic)
At the start: 0 parts

Commit message: Finished GPS
Parts:
- added C38, C40, C41: 100nF, symbol Device:C
- added C39: 10uF, symbol Device:C
- added J7: GPS antenna, symbol Connector:Conn_Coaxial
- added U8: MAX-M10S-00B, MAX-M10S-00B:XCVR_MAX-M10S-00B, symbol MAX-M10S-00B:MAX-M10S-00B
Connections:
- new net: J7.1 (In), U8.11 (RF_IN)
- new net +3V3: C38.2, C39.2, C40.2, C41.2, U8.6 (V_BCKP), U8.7 (V_IO), U8.8 (VCC)
- new net GND: C38.1, C39.1, C40.1, C41.1, J7.2 (Ext), U8.1 (GND), U8.10 (GND), U8.12 (GND)
- new net GPS_RX: U8.3 (RXD)
- new net GPS_TX: U8.2 (TXD)
- no-connect marks 0 -> 8
Other:
- note added: "Input:"
- note added: "Output:"
- note added: "Passive:"
