File: SSI Balloon Summer PCB/GPS.kicad_sch (KiCad schematic)
At the start: 6 parts, among them J7 GPS antenna, U8 MAX-M10S-00B

Commit message: Layout placement for every sheet except PWR and SD card
Parts:
- C38, C40, C41: footprint (none) -> Capacitor_SMD:C_0603_1608Metric
- C39: footprint (none) -> Capacitor_SMD:C_0805_2012Metric
- J7: footprint (none) -> Connector_Coaxial:U.FL_Hirose_U.FL-R-SMT-1_Vertical
Changed lines of the file:
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@@
 			)
 		)
-		(property "Footprint" ""
+		(property "Footprint" "Capacitor_SMD:C_0805_2012Metric"
 			(at 183.8452 73.66 0)
 			(hide yes)
@@
 			)
 		)
-		(property "Footprint" ""
+		(property "Footprint" "Capacitor_SMD:C_0603_1608Metric"
 			(at 172.4152 73.66 0)
 			(hide yes)
@@
 			)
 		)
-		(property "Footprint" ""
+		(property "Footprint" "Connector_Coaxial:U.FL_Hirose_U.FL-R-SMT-1_Vertical"
 			(at 97.79 99.06 0)
 			(hide yes)
@@
 			)
 		)
-		(property "Footprint" ""
+		(property "Footprint" "Capacitor_SMD:C_0603_1608Metric"
 			(at 178.1048 82.55 0)
 			(hide yes)
@@
 			)
 		)
-		(property "Footprint" ""
+		(property "Footprint" "Capacitor_SMD:C_0603_1608Metric"
 			(at 197.1548 80.01 0)
 			(hide yes)

Commit message: Reviewed sensor sheet
Parts:
- C38, C40, C41: footprint Capacitor_SMD:C_0603_1608Metric -> (none)
- C39: footprint Capacitor_SMD:C_0805_2012Metric -> (none)
- J7: footprint Connector_Coaxial:U.FL_Hirose_U.FL-R-SMT-1_Vertical -> (none)
Changed lines of the file:
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@@
 			)
 		)
-		(property "Footprint" "Capacitor_SMD:C_0805_2012Metric"
+		(property "Footprint" ""
 			(at 183.8452 73.66 0)
 			(hide yes)
@@
 			)
 		)
-		(property "Footprint" "Capacitor_SMD:C_0603_1608Metric"
+		(property "Footprint" ""
 			(at 172.4152 73.66 0)
 			(hide yes)
@@
 			)
 		)
-		(property "Footprint" "Connector_Coaxial:U.FL_Hirose_U.FL-R-SMT-1_Vertical"
+		(property "Footprint" ""
 			(at 97.79 99.06 0)
 			(hide yes)
@@
 			)
 		)
-		(property "Footprint" "Capacitor_SMD:C_0603_1608Metric"
+		(property "Footprint" ""
 			(at 178.1048 82.55 0)
 			(hide yes)
@@
 			)
 		)
-		(property "Footprint" "Capacitor_SMD:C_0603_1608Metric"
+		(property "Footprint" ""
 			(at 197.1548 80.01 0)
 			(hide yes)
