File: SSI Balloon Summer PCB/MCU.kicad_sch (KiCad schematic)
At the start: 18 parts, among them J5 Conn_01x05, SW2 SW_SPST, SW3 SW_SPST, U7 STM32F411CEUx, Y1 ABM8W-12.0000MHZ-8-K1Z-T3

Commit message: Finished sensors + tidied up schematic
Parts:
- added J9: Camera, symbol Connector_Generic:Conn_01x08
Connections:
- net GND: now also J9.5 (Pin_5)
- net MISO: now also J9.3 (Pin_3)
- net MOSI: now also J9.2 (Pin_2)
- net SCL: now also J9.8 (Pin_8)
- net SDA: now also J9.7 (Pin_7)
- net Cam_CS: now reaches U7.14 (PA4)
- net Cam_CS: now also J9.1 (Pin_1)
- net Temp_CS: now reaches U7.29 (PA8)
- net IMU_INT1: now reaches U7.38 (PA15)
- net BMP_CS renamed Baro_CS
- new net +5V: J9.6 (Pin_6)
- new net SCLK: J9.4 (Pin_4)
Other:
- note added: "Arducam Mini 2MP Plus, SKU B0067"
- moved on the sheet: C31, C32, R13, Y1

Commit message: tidying
Connections:
- net PI_ZERO_RX: no longer names the net of U7.33 (PA12)
- net PI_ZERO_TX: no longer names the net of U7.32 (PA11)
