File: SSI Balloon Summer PCB/Radio.kicad_sch (KiCad schematic)
At the start: 16 parts, among them J3 LoRa antenna, J4 APRS antenna, U1 RFM95W-915S2, U5 DRA818V

Commit message: stuff
Other:
- note added: "APRS_AUDIO unconnected so far"
Changed lines of the file:
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@@
 	(generator_version "10.0")
 	(paper "A4")
+	(text "APRS_AUDIO unconnected so far"
+		(exclude_from_sim no)
+		(at 165.354 69.088 0)
+		(effects
+			(font
+				(size 1.27 1.27)
+			)
+		)
+	)
 	(junction
 		(at 125.73 73.66)

Commit message: Added APRS_AUDIO
Changed lines of the file:
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@@
+	(wire
+		(pts
+			(xy 255.27 41.91) (xy 264.16 41.91)
+		)
+		(stroke
+			(width 0)
+			(type default)
+		)
+	)
 	(wire
 		(pts
@@
 	(label "LoRa_CS"
 		(at 255.27 33.02 180)
+		(effects
+			(font
+				(size 1.27 1.27)
+			)
+			(justify right bottom)
+		)
+	)
+	(label "APRS_AUDIO"
+		(at 255.27 41.91 180)
 		(effects
 			(font
@@
 		(effects
 			(font
+				(size 1.27 1.27)
+			)
+			(justify left)
+		)
+	)
+	(hierarchical_label "APRS_AUDIO"
+		(shape input)
+		(at 264.16 41.91 0)
+		(effects
+			(font
