File: SSI Balloon Summer PCB/SSI Flight Computer PCB/SSI Summer Balloons.kicad_sch (KiCad schematic)
At the start: 1 part, among them J10 Conn_01x08

Commit message: Various rewiring: SWD, microSD, APRS JST
Parts:
- added R11, R12: 10k, Resistor_SMD:R_0603_1608Metric, symbol Device:R
Connections:
- net +5V: now also J10.1 (Pin_1); no longer J10.8 (Pin_8)
- net GND: now also J10.2 (Pin_2), J10.3 (Pin_3); no longer J10.6 (Pin_6), J10.7 (Pin_7)
- net MCU (STM)/APRS_AUDIO: now also J10.4 (Pin_4); no longer J10.5 (Pin_5)
- net MCU (STM)/APRS_PD: now also J10.8 (Pin_8), R12.1; no longer J10.1 (Pin_1)
- net MCU (STM)/APRS_PTT: now also J10.7 (Pin_7), R11.1; no longer J10.2 (Pin_2)
- net MCU (STM)/APRS_RX: now also J10.6 (Pin_6); no longer J10.3 (Pin_3)
- net MCU (STM)/APRS_TX: now also J10.5 (Pin_5); no longer J10.4 (Pin_4)
- new net +3V3: R11.2, R12.2
Other:
- moved on the sheet: J10

Commit message: finished finding all parts on JLCPCB - finalizing BOM then order
Parts:
- J10: LCSC (none) -> C157914
- R11, R12: LCSC (none) -> C25804
Changed lines of the file:
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@@
+			)
+		)
+		(property "LCSC" "C157914"
+			(at 147.32 20.32 90)
+			(hide yes)
+			(show_name no)
+			(do_not_autoplace no)
+			(effects
+				(font
+					(size 1.27 1.27)
+				)
 			)
 		)
@@
 			)
 		)
+		(property "LCSC" "C25804"
+			(at 127 25.4 0)
+			(hide yes)
+			(show_name no)
+			(do_not_autoplace no)
+			(effects
+				(font
+					(size 1.27 1.27)
+				)
+			)
+		)
 		(pin "1"
 		)
@@
 			(at 119.38 29.21 0)
 			(hide yes)
+			(show_name no)
+			(do_not_autoplace no)
+			(effects
+				(font
+					(size 1.27 1.27)
+				)
+			)
+		)
+		(property "LCSC" "C25804"
+			(at 119.38 29.21 0)
+			(hide yes)
