File: SSI Balloon Summer PCB/SSI Flight Computer PCB/GPS.kicad_sch (KiCad schematic)
At the start: 6 parts, among them J7 GPS antenna, U8 MAX-M10S-00B

Commit message: Updated antenna connector
Parts:
- J7: footprint Connector_Coaxial:U.FL_Hirose_U.FL-R-SMT-1_Vertical -> Connector_Coaxial:SMA_Amphenol_901-144_Vertical
Changed lines of the file:
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@@
 			)
 		)
-		(property "Footprint" "Connector_Coaxial:U.FL_Hirose_U.FL-R-SMT-1_Vertical"
+		(property "Footprint" "Connector_Coaxial:SMA_Amphenol_901-144_Vertical"
 			(at 97.79 99.06 0)
 			(hide yes)

Commit message: finished finding all parts on JLCPCB - finalizing BOM then order
Parts:
- C38, C40, C41: LCSC (none) -> C519438
- C39: LCSC (none) -> C5189822
- J7: LCSC (none) -> C376663
- U8: LCSC (none) -> C4153167
Changed lines of the file:
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@@
+			)
+		)
+		(property "LCSC" "C5189822"
+			(at 182.88 69.85 0)
+			(hide yes)
+			(show_name no)
+			(do_not_autoplace no)
+			(effects
+				(font
+					(size 1.27 1.27)
+				)
 			)
 		)
@@
 			)
 		)
+		(property "LCSC" "C519438"
+			(at 171.45 69.85 0)
+			(hide yes)
+			(show_name no)
+			(do_not_autoplace no)
+			(effects
+				(font
+					(size 1.27 1.27)
+				)
+			)
+		)
 		(pin "2"
 		)
@@
 			)
 		)
-		(property "Datasheet" ""
+		(property "Datasheet" "HAND SOLDER THIS"
 			(at 97.79 99.06 0)
 			(hide yes)
@@
 		)
 		(property "PART_REV" ""
+			(at 97.79 99.06 90)
+			(hide yes)
+			(show_name no)
+			(do_not_autoplace no)
+			(effects
+				(font
+					(size 1.27 1.27)
+				)
+			)
+		)
+		(property "LCSC" "C376663"
 			(at 97.79 99.06 90)
 			(hide yes)
@@
 			)
 		)
+		(property "LCSC" "C519438"
+			(at 204.47 95.25 0)
+			(hide yes)
+			(show_name no)
+			(do_not_autoplace no)
+			(effects
+				(font
+					(size 1.27 1.27)
+				)
+			)
+		)
 		(pin "2"
 		)
@@
 			)
 		)
+		(property "LCSC" "C519438"
+			(at 222.25 83.82 0)
+			(hide yes)
+			(show_name no)
+			(do_not_autoplace no)
+			(effects
+				(font
+					(size 1.27 1.27)
+				)
+			)
+		)
 		(pin "2"
 		)
@@
 			(at 146.05 92.71 0)
 			(hide yes)
+			(show_name no)
+			(do_not_autoplace no)
+			(effects
+				(font
+					(size 1.27 1.27)
+				)
+			)
+		)
+		(property "LCSC" "C4153167"
+			(at 146.05 92.71 0)
+			(hide yes)

Commit message: PCB finally done i think and ready to order
Parts:
- C38, C40, C41: LCSC C519438 -> C14663
- C39: LCSC C5189822 -> C15850
Changed lines of the file:
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@@
 			)
 		)
-		(property "LCSC" "C5189822"
+		(property "LCSC" "C15850"
 			(at 182.88 69.85 0)
 			(hide yes)
@@
 			)
 		)
-		(property "LCSC" "C519438"
+		(property "LCSC" "C14663"
 			(at 171.45 69.85 0)
 			(hide yes)
@@
 			)
 		)
-		(property "LCSC" "C519438"
+		(property "LCSC" "C14663"
 			(at 204.47 95.25 0)
 			(hide yes)
@@
 			)
 		)
-		(property "LCSC" "C519438"
+		(property "LCSC" "C14663"
 			(at 222.25 83.82 0)
 			(hide yes)

Commit message: Board done but we have a price crisis so might have to change things
Parts:
- J7: now not fitted; now left out of the parts list
Changed lines of the file:
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@@
 		(body_style 1)
 		(exclude_from_sim no)
-		(in_bom yes)
+		(in_bom no)
 		(on_board yes)
 		(in_pos_files yes)
-		(dnp no)
+		(dnp yes)
 		(fields_autoplaced yes)
 		(property "Reference" "J7"
