File: SSI Balloon Summer PCB/SSI Flight Computer PCB/Sensor.kicad_sch (KiCad schematic)
At the start: 16 parts, among them J8 PT1000 Sensor, U10 MS5611-01BA03, U4 ICM-42688-P, U9 MAX31865ATP_T

Commit message: Cleaned APRS Filter up and adding Testing points
Parts:
- added TP11, TP8: TestPoint, TestPoint:TestPoint_Pad_1.5x1.5mm, symbol Connector:TestPoint
Connections:
- net GND: now also TP8.1
- net IMU_INT1: now also TP11.1

Commit message: Added Headers for testing, finalizing PCB
Parts:
- removed TP11, TP8: TestPoint, TestPoint:TestPoint_Pad_1.5x1.5mm, symbol Connector:TestPoint
- added TP11, TP20, TP21, TP22, TP8: Conn_01x01, Connector_PinHeader_2.54mm:PinHeader_1x01_P2.54mm_Vertical, symbol Connector_Generic:Conn_01x01
Connections:
- net BARO_CS: now also TP22.1 (Pin_1)
- net GND: now also TP8.1 (Pin_1)
- net IMU_CS: now also TP20.1 (Pin_1)
- net IMU_INT1: now also TP11.1 (Pin_1)
- net Temp_CS: now also TP21.1 (Pin_1)

Commit message: More silkscreen organization, combined some pinheaders
Parts:
- TP11: value Conn_01x01 -> IMU_INT1
- TP20: value Conn_01x01 -> IMU_CS
- TP21: value Conn_01x01 -> Temp_CS
- TP22: value Conn_01x01 -> BARO_CS
- TP8: value Conn_01x01 -> GND
Changed lines of the file:
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@@
 			)
 		)
-		(property "Value" "Conn_01x01"
+		(property "Value" "GND"
 			(at 143.51 40.6399 0)
 			(show_name no)
@@
 			)
 		)
-		(property "Value" "Conn_01x01"
+		(property "Value" "Temp_CS"
 			(at 63.5 52.0699 0)
 			(show_name no)
@@
 			)
 		)
-		(property "Value" "Conn_01x01"
+		(property "Value" "IMU_INT1"
 			(at 91.44 39.3699 0)
 			(show_name no)
@@
 			)
 		)
-		(property "Value" "Conn_01x01"
+		(property "Value" "IMU_CS"
 			(at 62.23 39.3699 0)
 			(show_name no)
@@
 			)
 		)
-		(property "Value" "Conn_01x01"
+		(property "Value" "BARO_CS"
 			(at 96.52 52.0699 0)
 			(show_name no)

Commit message: finished finding all parts on JLCPCB - finalizing BOM then order
Parts:
- C11: value 0.1uF -> 100nF; LCSC (none) -> C519438
- C12: LCSC (none) -> C43922
- C42: LCSC (none) -> C36911415
- C43, C44, C46: LCSC (none) -> C519438
- C45: LCSC (none) -> C49326291
- J8: LCSC (none) -> C158004
- R21: LCSC (none) -> C2989227
- R22: LCSC (none) -> C7250
- R23, R24, R25: LCSC (none) -> C25804
- TP11, TP20, TP21, TP22, TP8: LCSC (none) -> C81276
- U10: LCSC (none) -> C15639
- U4: LCSC (none) -> C1850418
- U9: LCSC (none) -> C118474

Commit message: PCB finally done i think and ready to order
Parts:
- added R31: 1k, Resistor_SMD:R_0603_1608Metric, symbol Device:R
- C11, C43, C44, C46: LCSC C519438 -> C14663
- C42: LCSC C36911415 -> C163179
Connections:
- net GND: now also R31.1; no longer U4.9 (INT2/FSYNC/CLKIN)
- new net: R31.2, U4.9 (INT2/FSYNC/CLKIN)
Changed lines of the file:
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@@
 	(wire
 		(pts
+			(xy 36.83 87.63) (xy 36.83 91.44)
+		)
+		(stroke
+			(width 0)
+			(type default)
+		)
+	)
+	(wire
+		(pts
 			(xy 228.6 92.71) (xy 236.22 92.71)
 		)
@@
 	(wire
 		(pts
+			(xy 36.83 77.47) (xy 36.83 80.01)
+		)
+		(stroke
+			(width 0)
+			(type default)
+		)
+	)
+	(wire
+		(pts
 			(xy 30.48 96.52) (xy 35.56 96.52)
 		)
@@
 			)
 		)
-		(property "LCSC" "C519438"
+		(property "LCSC" "C14663"
 			(at 104.14 77.47 0)
 			(hide yes)
@@
 	)
 	(symbol
-		(lib_id "power:+3V3")
-		(at 35.56 107.95 180)
+		(lib_id "Device:R")
+		(at 36.83 83.82 0)
 		(unit 1)
 		(body_style 1)
@@
 		(in_pos_files yes)
 		(dnp no)
-		(fields_autoplaced yes)
-		(property "Reference" "#PWR0105"
-			(at 35.56 104.14 0)
-			(hide yes)
+		(property "Reference" "R31"
+			(at 34.29 83.82 90)
 			(show_name no)
 			(do_not_autoplace no)
@@
 			)
 		)
-		(property "Value" "+3V3"
-			(at 35.56 113.03 0)
+		(property "Value" "1k"
+			(at 31.75 83.82 90)
 			(show_name no)
 			(do_not_autoplace no)
@@
 			)
 		)
-		(property "Footprint" ""
-			(at 35.56 107.95 0)
+		(property "Footprint" "Resistor_SMD:R_0603_1608Metric"
+			(at 35.052 83.82 90)
 			(hide yes)
 			(show_name no)
@@
 		)
 		(property "Datasheet" ""
-			(at 35.56 107.95 0)
+			(at 36.83 83.82 0)
 			(hide yes)
 			(show_name no)
@@
 			)
 		)
-		(property "Description" "Power symbol creates a global label with name \"+3V3\""
-			(at 35.56 107.95 0)
+		(property "Description" "Resistor"
+			(at 36.83 83.82 0)
+			(hide yes)
+			(show_name no)
+			(do_not_autoplace no)
+			(effects
+				(font
+					(size 1.27 1.27)
+				)
+			)
+		)
+		(property "PART_REV" ""
+			(at 36.83 83.82 90)
+			(hide yes)
+			(show_name no)
+			(do_not_autoplace no)
+			(effects
+				(font
+					(size 1.27 1.27)
+				)
+			)
+		)
+		(property "LCSC" "C21190"
+			(at 36.83 83.82 90)
 			(hide yes)
 			(show_name no)
@@
 		(pin "1"
 		)
+		(pin "2"
+		)
 		(instances
 			(project "SSI Summer Balloons"
 				(path "/3c45a535-6e6b-4825-ad52-82c10cbe7866/98c67578-63cf-4cdd-a22b-0d2ebd53e276"
-					(reference "#PWR0105")
+					(reference "R31")
 					(unit 1)
 				)
@@
 	)
 	(symbol
-		(lib_id "Connector_Generic:Conn_01x01")
-		(at 88.9 38.1 0)
+		(lib_id "power:+3V3")
+		(at 35.56 107.95 180)
 		(unit 1)
 		(body_style 1)
@@
 		(dnp no)
 		(fields_autoplaced yes)
-		(property "Reference" "TP11"
-			(at 91.44 36.8299 0)
-			(show_name no)
-			(do_not_autoplace no)
-			(effects
-				(font
-					(size 1.27 1.27)
-				)
-				(justify left)
-			)
-		)
-		(property "Value" "IMU_INT1"
-			(at 91.44 39.3699 0)
+		(property "Reference" "#PWR0105"
+			(at 35.56 104.14 0)
+			(hide yes)
 			(show_name no)
 			(do_not_autoplace no)
@@
 					(size 1.27 1.27)
 				)
-				(justify left)
 			)
 		)
-		(property "Footprint" "Connector_PinHeader_2.54mm:PinHeader_1x01_P2.54mm_Vertical"
-			(at 88.9 38.1 0)
-			(hide yes)
+		(property "Value" "+3V3"
+			(at 35.56 113.03 0)
 			(show_name no)
 			(do_not_autoplace no)
@@
 			)
 		)
-		(property "Datasheet" "C81276"
-			(at 88.9 38.1 0)
+		(property "Footprint" ""
+			(at 35.56 107.95 0)
 			(hide yes)
 			(show_name no)
@@
 			)
 		)
-		(property "Description" "Generic connector, single row, 01x01, script generated (kicad-library-utils/schlib/autogen/connector/)"
-			(at 88.9 38.1 0)
+		(property "Datasheet" ""
+			(at 35.56 107.95 0)
 			(hide yes)
 			(show_name no)
@@
 			)
 		)
-		(property "LCSC" "C81276"
-			(at 88.9 38.1 0)
+		(property "Description" "Power symbol creates a global label with name \"+3V3\""
+			(at 35.56 107.95 0)
 			(hide yes)
 			(show_name no)
@@
 			(project "SSI Summer Balloons"
 				(path "/3c45a535-6e6b-4825-ad52-82c10cbe7866/98c67578-63cf-4cdd-a22b-0d2ebd53e276"
-					(reference "TP11")
+					(reference "#PWR0105")
 					(unit 1)
 				)
@@
 	)
 	(symbol
-		(lib_id "power:GND")
-		(at 251.46 83.82 0)
+		(lib_id "Connector_Generic:Conn_01x01")
+		(at 88.9 38.1 0)
 		(unit 1)
 		(body_style 1)
@@
 		(dnp no)
 		(fields_autoplaced yes)
-		(property "Reference" "#PWR091"
-			(at 251.46 90.17 0)
-			(hide yes)
+		(property "Reference" "TP11"
+			(at 91.44 36.8299 0)
 			(show_name no)
 			(do_not_autoplace no)
@@
 					(size 1.27 1.27)
 				)
+				(justify left)
 			)
 		)
-		(property "Value" "GND"
-			(at 251.46 88.9 0)
+		(property "Value" "IMU_INT1"
+			(at 91.44 39.3699 0)
 			(show_name no)
 			(do_not_autoplace no)
@@
 					(size 1.27 1.27)
 				)
+				(justify left)
 			)
 		)
-		(property "Footprint" ""
-			(at 251.46 83.82 0)
+		(property "Footprint" "Connector_PinHeader_2.54mm:PinHeader_1x01_P2.54mm_Vertical"
+			(at 88.9 38.1 0)
 			(hide yes)
 			(show_name no)
@@
 			)
 		)
-		(property "Datasheet" ""
-			(at 251.46 83.82 0)
+		(property "Datasheet" "C81276"
+			(at 88.9 38.1 0)
 			(hide yes)
 			(show_name no)
@@
 			)
 		)
-		(property "Description" "Power symbol creates a global label with name \"GND\" , ground"
-			(at 251.46 83.82 0)
+		(property "Description" "Generic connector, single row, 01x01, script generated (kicad-library-utils/schlib/autogen/connector/)"
+			(at 88.9 38.1 0)
+			(hide yes)
+			(show_name no)
+			(do_not_autoplace no)
+			(effects
+				(font
+					(size 1.27 1.27)
+				)
+			)
+		)
+		(property "LCSC" "C81276"
+			(at 88.9 38.1 0)
 			(hide yes)
 			(show_name no)
@@
 			(project "SSI Summer Balloons"
 				(path "/3c45a535-6e6b-4825-ad52-82c10cbe7866/98c67578-63cf-4cdd-a22b-0d2ebd53e276"
-					(reference "#PWR091")
+					(reference "TP11")
 					(unit 1)
 				)
@@
 	(symbol
 		(lib_id "power:GND")
-		(at 36.83 91.44 180)
+		(at 251.46 83.82 0)
 		(unit 1)
 		(body_style 1)
@@
 		(dnp no)
 		(fields_autoplaced yes)
-		(property "Reference" "#PWR020"
-			(at 36.83 85.09 0)
+		(property "Reference" "#PWR091"
+			(at 251.46 90.17 0)
 			(hide yes)
 			(show_name no)
@@
 		)
 		(property "Value" "GND"
-			(at 39.37 90.1699 0)
+			(at 251.46 88.9 0)
 			(show_name no)
 			(do_not_autoplace no)
@@
 					(size 1.27 1.27)
 				)
-				(justify right)
 			)
 		)
 		(property "Footprint" ""
-			(at 36.83 91.44 0)
+			(at 251.46 83.82 0)
 			(hide yes)
 			(show_name no)
@@
 		)
 		(property "Datasheet" ""
-			(at 36.83 91.44 0)
+			(at 251.46 83.82 0)
 			(hide yes)
 			(show_name no)
@@
 		)
 		(property "Description" "Power symbol creates a global label with name \"GND\" , ground"
-			(at 36.83 91.44 0)
+			(at 251.46 83.82 0)
 			(hide yes)
 			(show_name no)
@@
 			(project "SSI Summer Balloons"
 				(path "/3c45a535-6e6b-4825-ad52-82c10cbe7866/98c67578-63cf-4cdd-a22b-0d2ebd53e276"
-					(reference "#PWR020")
+					(reference "#PWR091")
 					(unit 1)
 				)
@@
 			)
 		)
-		(property "LCSC" "C519438"
+		(property "LCSC" "C14663"
 			(at 151.13 137.16 0)
 			(hide yes)
@@
 			)
 		)
-		(property "LCSC" "C519438"
+		(property "LCSC" "C14663"
 			(at 224.79 57.15 0)
 			(hide yes)
@@
 	)
 	(symbol
+		(lib_id "power:GND")
+		(at 36.83 77.47 180)
+		(unit 1)
+		(body_style 1)
+		(exclude_from_sim no)
+		(in_bom yes)
+		(on_board yes)
+		(in_pos_files yes)
+		(dnp no)
+		(fields_autoplaced yes)
+		(property "Reference" "#PWR020"
+			(at 36.83 71.12 0)
+			(hide yes)
+			(show_name no)
+			(do_not_autoplace no)
+			(effects
+				(font
+					(size 1.27 1.27)
+				)
+			)
+		)
+		(property "Value" "GND"
+			(at 36.83 72.39 0)
+			(show_name no)
+			(do_not_autoplace no)
+			(effects
+				(font
+					(size 1.27 1.27)
+				)
+			)
+		)
+		(property "Footprint" ""
+			(at 36.83 77.47 0)
+			(hide yes)
+			(show_name no)
+			(do_not_autoplace no)
+			(effects
+				(font
+					(size 1.27 1.27)
+				)
+			)
+		)
+		(property "Datasheet" ""
+			(at 36.83 77.47 0)
+			(hide yes)
+			(show_name no)
+			(do_not_autoplace no)
+			(effects
+				(font
+					(size 1.27 1.27)
+				)
+			)
+		)
+		(property "Description" "Power symbol creates a global label with name \"GND\" , ground"
+			(at 36.83 77.47 0)
+			(hide yes)
+			(show_name no)
+			(do_not_autoplace no)
+			(effects
+				(font
+					(size 1.27 1.27)
+				)
+			)
+		)
+		(pin "1"
+		)
+		(instances
+			(project "SSI Summer Balloons"
+				(path "/3c45a535-6e6b-4825-ad52-82c10cbe7866/98c67578-63cf-4cdd-a22b-0d2ebd53e276"
+					(reference "#PWR020")
+					(unit 1)
+				)
+			)
+		)
+	)
+	(symbol
 		(lib_id "Device:C")
 		(at 158.75 97.79 0)
@@
 			)
 		)
-		(property "LCSC" "C519438"
+		(property "LCSC" "C14663"
 			(at 251.46 77.47 0)
 			(hide yes)
@@
 			)
 		)
-		(property "LCSC" "C36911415"
+		(property "LCSC" "C163179"
 			(at 123.19 91.44 0)
 			(hide yes)

Commit message: Board done but we have a price crisis so might have to change things
Parts:
- C42: LCSC C163179 -> C57112
- C45: LCSC C49326291 -> C57112
- TP11, TP20, TP21, TP22, TP8: now not fitted; now left out of the parts list
Changed lines of the file:
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@@
 		(body_style 1)
 		(exclude_from_sim no)
-		(in_bom yes)
+		(in_bom no)
 		(on_board yes)
 		(in_pos_files yes)
-		(dnp no)
+		(dnp yes)
 		(fields_autoplaced yes)
 		(property "Reference" "TP8"
@@
 		(body_style 1)
 		(exclude_from_sim no)
-		(in_bom yes)
+		(in_bom no)
 		(on_board yes)
 		(in_pos_files yes)
-		(dnp no)
+		(dnp yes)
 		(fields_autoplaced yes)
 		(property "Reference" "TP21"
@@
 		(body_style 1)
 		(exclude_from_sim no)
-		(in_bom yes)
+		(in_bom no)
 		(on_board yes)
 		(in_pos_files yes)
-		(dnp no)
+		(dnp yes)
 		(fields_autoplaced yes)
 		(property "Reference" "TP11"
@@
 			)
 		)
-		(property "LCSC" "C49326291"
+		(property "LCSC" "C57112"
 			(at 158.75 97.79 0)
 			(hide yes)
@@
 		(body_style 1)
 		(exclude_from_sim no)
-		(in_bom yes)
+		(in_bom no)
 		(on_board yes)
 		(in_pos_files yes)
-		(dnp no)
+		(dnp yes)
 		(fields_autoplaced yes)
 		(property "Reference" "TP20"
@@
 		(body_style 1)
 		(exclude_from_sim no)
-		(in_bom yes)
+		(in_bom no)
 		(on_board yes)
 		(in_pos_files yes)
-		(dnp no)
+		(dnp yes)
 		(fields_autoplaced yes)
 		(property "Reference" "TP22"
@@
 			)
 		)
-		(property "LCSC" "C163179"
+		(property "LCSC" "C57112"
 			(at 123.19 91.44 0)
 			(hide yes)
