File: SSI Balloon Summer PCB/SSI APRS/SSI APRS.kicad_sch (KiCad schematic)
At the start: 31 parts, among them J1 Conn_01x08, J4 APRS antenna, U12 TPS63070RNMR, U5 DRA818V

Commit message: Board done but we have a price crisis so might have to change things
Parts:
- C17, C18: LCSC C344022 -> C96446
- C20, C21, C22: LCSC C48986262 -> C45783
- J4: LCSC C376663 -> (none); now not fitted; now left out of the parts list
- R20B1: now left out of the parts list
- TP1, TP2, TP3, TP4, TP5, TP6, TP7: now not fitted; now left out of the parts list
- U5: now not fitted
Changed lines of the file:
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@@
 			)
 		)
-		(property "LCSC" "C48986262"
+		(property "LCSC" "C45783"
 			(at 121.92 78.74 0)
 			(hide yes)
@@
 		(body_style 1)
 		(exclude_from_sim no)
-		(in_bom yes)
+		(in_bom no)
 		(on_board yes)
 		(in_pos_files yes)
-		(dnp no)
+		(dnp yes)
 		(fields_autoplaced yes)
 		(property "Reference" "TP7"
@@
 		(body_style 1)
 		(exclude_from_sim no)
-		(in_bom yes)
+		(in_bom no)
 		(on_board yes)
 		(in_pos_files yes)
-		(dnp no)
+		(dnp yes)
 		(fields_autoplaced yes)
 		(property "Reference" "TP1"
@@
 		(body_style 1)
 		(exclude_from_sim no)
-		(in_bom yes)
+		(in_bom no)
 		(on_board yes)
 		(in_pos_files yes)
-		(dnp no)
+		(dnp yes)
 		(fields_autoplaced yes)
 		(property "Reference" "TP2"
@@
 			)
 		)
-		(property "LCSC" "C48986262"
+		(property "LCSC" "C45783"
 			(at 129.54 78.74 0)
 			(hide yes)
@@
 		(body_style 1)
 		(exclude_from_sim no)
-		(in_bom yes)
+		(in_bom no)
 		(on_board yes)
 		(in_pos_files yes)
-		(dnp no)
+		(dnp yes)
 		(fields_autoplaced yes)
 		(property "Reference" "J4"
@@
 			)
 		)
-		(property "LCSC" "C376663"
+		(property "LCSC" ""
 			(at 215.9 128.27 90)
 			(hide yes)
@@
 		(body_style 1)
 		(exclude_from_sim no)
-		(in_bom yes)
+		(in_bom no)
 		(on_board yes)
 		(in_pos_files yes)
@@
 		(on_board yes)
 		(in_pos_files yes)
-		(dnp no)
+		(dnp yes)
 		(fields_autoplaced yes)
 		(property "Reference" "U5"
@@
 			)
 		)
-		(property "LCSC" "C344022"
+		(property "LCSC" "C96446"
 			(at 99.06 78.74 0)
 			(hide yes)
@@
 			)
 		)
-		(property "LCSC" "C344022"
+		(property "LCSC" "C96446"
 			(at 57.15 78.74 0)
 			(hide yes)
@@
 			)
 		)
-		(property "LCSC" "C48986262"
+		(property "LCSC" "C45783"
 			(at 137.16 78.74 0)
 			(hide yes)
@@
 		(body_style 1)
 		(exclude_from_sim no)
-		(in_bom yes)
+		(in_bom no)
 		(on_board yes)
 		(in_pos_files yes)
-		(dnp no)
+		(dnp yes)
 		(fields_autoplaced yes)
 		(property "Reference" "TP6"
@@
 		(body_style 1)
 		(exclude_from_sim no)
-		(in_bom yes)
+		(in_bom no)
 		(on_board yes)
 		(in_pos_files yes)
-		(dnp no)
+		(dnp yes)
 		(fields_autoplaced yes)
 		(property "Reference" "TP5"
@@
 		(body_style 1)
 		(exclude_from_sim no)
-		(in_bom yes)
+		(in_bom no)
 		(on_board yes)
 		(in_pos_files yes)
-		(dnp no)
+		(dnp yes)
 		(fields_autoplaced yes)
 		(property "Reference" "TP3"
@@
 		(body_style 1)
 		(exclude_from_sim no)
-		(in_bom yes)
+		(in_bom no)
 		(on_board yes)
 		(in_pos_files yes)
-		(dnp no)
+		(dnp yes)
 		(fields_autoplaced yes)
 		(property "Reference" "TP4"
